File: Alexandrie.sch (KiCad schematic (older format))
At the start: 47 parts, among them J1 kk_10, J11 CONN_01X03, J2 kk_5, J3 kk_5, J4 CONN_01X06, J5 CONN_01X02, J6 CONN_01X13, J7 CONN_01X06, J8 kk_10, U1 74HCT04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

Commit message: minor changes, BOM added
Parts:
- U12: value LD29150DT50R -> 78M05 Dpak

Commit message: new gerber, minor mods
Parts:
- removed J7: CONN_01X06, conn_kk100:kk100_22-23-2061, symbol CONN_01X06
- added J7: Conn_01x07, Connectors_Molex:Molex_KK-6410-07_07x2.54mm_Straight, symbol Conn_01x07
Connections:
- net +12V: now also J7.7 (Pin_7)
- net GND: now also J7.6 (Pin_6)
- net RX2_IN: now also J7.4 (Pin_4)
- net RX3_IN: now also J7.3 (Pin_3)
- net RX_BYPASS_OUT: now also J7.2 (Pin_2)
- net TX_RX_RLY: now also J7.1 (Pin_1)
- net Xvtr_IN: now also J7.5 (Pin_5)
Other:
- moved on the sheet: J3
Changed lines of the file:
@@
 L CONN_01X05 J3
 U 1 1 5939C57F
-P 10650 3600
-F 0 "J3" H 10650 3900 50  0000 C CNN
-F 1 "kk_5" V 10750 3600 50  0000 C CNN
-F 2 "conn_kk100:kk100_22-23-2051" H 10650 3600 50  0001 C CNN
-F 3 "" H 10650 3600 50  0001 C CNN
-	1    10650 3600
+P 10650 3700
+F 0 "J3" H 10650 4000 50  0000 C CNN
+F 1 "kk_5" V 10750 3700 50  0000 C CNN
+F 2 "conn_kk100:kk100_22-23-2051" H 10650 3700 50  0001 C CNN
+F 3 "" H 10650 3700 50  0001 C CNN
+	1    10650 3700
 	1    0    0    1
 $EndComp
@@
 L GND #PWR058
 U 1 1 5939C585
+P 10400 3600
+F 0 "#PWR058" H 10400 3350 50  0001 C CNN
+F 1 "GND" V 10450 3650 20  0000 C CNN
+F 2 "" H 10400 3600 50  0001 C CNN
+F 3 "" H 10400 3600 50  0001 C CNN
+	1    10400 3600
+	0    1    -1   0
+$EndComp
+$Comp
+L +12V #PWR059
+U 1 1 5939C58B
 P 10400 3500
-F 0 "#PWR058" H 10400 3250 50  0001 C CNN
-F 1 "GND" V 10450 3550 20  0000 C CNN
+F 0 "#PWR059" H 10400 3350 50  0001 C CNN
+F 1 "+12V" V 10400 3700 50  0000 C CNN
 F 2 "" H 10400 3500 50  0001 C CNN
 F 3 "" H 10400 3500 50  0001 C CNN
 	1    10400 3500
-	0    1    -1   0
-$EndComp
-$Comp
-L +12V #PWR059
-U 1 1 5939C58B
-P 10400 3400
-F 0 "#PWR059" H 10400 3250 50  0001 C CNN
-F 1 "+12V" V 10400 3600 50  0000 C CNN
-F 2 "" H 10400 3400 50  0001 C CNN
-F 3 "" H 10400 3400 50  0001 C CNN
-	1    10400 3400
 	0    -1   1    0
 $EndComp
@@
 Text GLabel 5300 2700 2    39   Input ~ 0
 Ant_3
-Text GLabel 10400 3600 0    39   Input ~ 0
+Text GLabel 10400 3700 0    39   Input ~ 0
 Ant_1
-Text GLabel 10400 3700 0    39   Input ~ 0
+Text GLabel 10400 3800 0    39   Input ~ 0
 Ant_2
-Text GLabel 10400 3800 0    39   Input ~ 0
+Text GLabel 10400 3900 0    39   Input ~ 0
 Ant_3
 Text Notes 10500 4350 2    39   ~ 0
@@
 $EndComp
 $Comp
-L CONN_01X06 J7
-U 1 1 59411EA5
-P 10650 2950
-F 0 "J7" H 10650 3300 50  0000 C CNN
-F 1 "CONN_01X06" V 10750 2950 50  0000 C CNN
-F 2 "conn_kk100:kk100_22-23-2061" H 10650 2950 50  0001 C CNN
-F 3 "" H 10650 2950 50  0001 C CNN
-	1    10650 2950
-	1    0    0    1
-$EndComp
-$Comp
 L +5V #PWR062
 U 1 1 593D3009
@@
 	10400 2800 10450 2800
 Wire Wire Line
-	10400 3400 10450 3400
-Wire Wire Line
 	10400 3500 10450 3500
 Wire Wire Line
+	10400 3600 10450 3600
+Wire Wire Line
+	10400 3900 10450 3900
+Wire Wire Line
 	10400 3800 10450 3800
 Wire Wire Line
 	10400 3700 10450 3700
-Wire Wire Line
-	10400 3600 10450 3600
 Wire Wire Line
 	4200 1350 4200 3050
@@
 Wire Wire Line
 	2000 750  2000 1000
+Text GLabel 10200 3300 0    39   Input ~ 0
+TX_RX_RLY
+Wire Wire Line
+	10450 3300 10200 3300
+$Comp
+L Conn_01x07 J7
+U 1 1 5A61D7BF
+P 10650 3000
+F 0 "J7" H 10650 3400 50  0000 C CNN
+F 1 "Conn_01x07" H 10650 2600 50  0000 C CNN
+F 2 "Connectors_Molex:Molex_KK-6410-07_07x2.54mm_Straight" H 10650 3000 50  0001 C CNN
+F 3 "" H 10650 3000 50  0001 C CNN
+	1    10650 3000
+	1    0    0    1
+$EndComp
 $EndSCHEMATC

Commit message: stable V2.0
Connections:
- net +12V: now also C17.1; no longer C17.2
- net +5V: now also C19.1; no longer C19.2
- net GND: now also C17.2, C19.2; no longer C17.1, C19.1
Other:
- note added: "Jaune"
- note added: "jaune\n"
- note added: "rouge"
- note added: "rouge\n"
Changed lines of the file:
@@
 EESchema Schematic File Version 2
 LIBS:Alexandrie-rescue
-LIBS:power
-LIBS:device
-LIBS:conn
-LIBS:regul
-LIBS:74xx
 LIBS:7805d-pack
 LIBS:tpic6b595
+LIBS:Connector_Generic
+LIBS:Device
+LIBS:power
+LIBS:Regulator_Linear
 LIBS:Alexandrie-cache
 EELAYER 25 0
@@
 F 3 "" H 7750 5500 50  0001 C CNN
 	1    7750 5500
-	0    1    1    0
+	0    -1   -1   0
 $EndComp
 $Comp
@@
 F 3 "" H 7750 4450 50  0001 C CNN
 	1    7750 4450
-	0    1    1    0
+	0    -1   -1   0
 $EndComp
 $Comp
@@
 	1    0    0    1
 $EndComp
+Text Notes 5700 3100 0    100  ~ 20
+rouge
+Text Notes 5700 1400 0    100  ~ 20
+jaune\n
+Text Notes 5300 4400 1    100  ~ 20
+Jaune
+Text Notes 6550 5800 1    100  ~ 20
+rouge\n
 $EndSCHEMATC
