File: Alexandrie.sch (KiCad schematic (older format))
At the start: 47 parts, among them J1 kk_10, J11 CONN_01X03, J2 kk_5, J3 kk_5, J4 CONN_01X06, J5 CONN_01X02, J6 CONN_01X13, J7 Conn_01x07, J8 kk_10, U1 74HCT04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

Commit message: cleaning, new bom and interactive bom
Other:
- note added: "To\nThemis\nBoard"
- note removed: "To\nVSWR/PS/TX-RX \nBoard"
Changed lines of the file:
@@
 EESchema Schematic File Version 4
 LIBS:Alexandrie-cache
-EELAYER 26 0
+EELAYER 29 0
 EELAYER END
 $Descr A4 11693 8268
@@
 TX_RX_RLY
 Text Notes 3200 1850 0    39   ~ 8
-To\nVSWR/PS/TX-RX \nBoard
+To\nThemis\nBoard
 Text Notes 3550 1250 0    20   ~ 0
 <--\nFWD
